File: Open2327RomAdapter.sch (KiCad schematic (older format))
At the start: 5 parts, among them P1 CONN_01X02, SW1 SW_SPST, U1 2364, U2 27128

Commit message: Add pull-up resistors
Parts:
- removed P1: CONN_01X02, Sukko:LoosePads-2, symbol CONN_01X02
- removed SW1: SW_SPST, symbol SW_SPST-RESCUE-Open2327RomAdapter
- added P1: Conn_01x04, symbol Conn_01x04
- added R2, R3: 10K, Resistors_SMD:R_0805_HandSoldering, symbol R
Connections:
- wire segments 105 -> 111
Other:
- moved on the sheet: R1

Commit message: Update board This should be the board that went to prototype production. It has been tested and is working great!
Parts:
- P1: value Conn_01x04 -> CONN_01X04; footprint (none) -> Sukko:LoosePads-4
- U1: footprint Housings_DIP:DIP-24_W15.24mm -> Open2327RomAdapter:DIP-24_W15.24mm-Notch
- U2: footprint Housings_DIP:DIP-28_W15.24mm -> Open2327RomAdapter:DIP-28_W15.24mm-Notch
Changed lines of the file:
@@
 F 0 "U1" H 5400 4250 60  0000 C CNN
 F 1 "2364" H 5400 5650 60  0000 C CNN
-F 2 "Housings_DIP:DIP-24_W15.24mm" H 5400 5650 60  0001 C CNN
+F 2 "Open2327RomAdapter:DIP-24_W15.24mm-Notch" H 5400 5650 60  0001 C CNN
 F 3 "" H 5400 5650 60  0001 C CNN
 	1    5400 4950
@@
 F 0 "U2" H 5450 3050 50  0000 C CNN
 F 1 "27128" H 6000 1050 50  0000 C CNN
-F 2 "Housings_DIP:DIP-28_W15.24mm" H 5700 2050 50  0001 C CNN
+F 2 "Open2327RomAdapter:DIP-28_W15.24mm-Notch" H 5700 2050 50  0001 C CNN
 F 3 "" H 5700 2050 50  0000 C CNN
 	1    5700 2050
@@
 P 4400 3300
 F 0 "P1" V 4500 3250 50  0000 C CNN
-F 1 "Conn_01x04" V 4400 3000 50  0001 C CNN
-F 2 "" H 4400 3300 50  0001 C CNN
+F 1 "CONN_01X04" V 4400 3000 50  0001 C CNN
+F 2 "Sukko:LoosePads-4" H 4400 3300 50  0001 C CNN
 F 3 "" H 4400 3300 50  0001 C CNN
 	1    4400 3300

Commit message: Cleanup
Parts:
- P1: footprint Sukko:LoosePads-4 -> Open2327RomAdapter:LoosePads-4
Changed lines of the file:
@@
 EESchema Schematic File Version 2
-LIBS:Open2327RomAdapter-rescue
 LIBS:power
 LIBS:device
@@
 F 0 "P1" V 4500 3250 50  0000 C CNN
 F 1 "CONN_01X04" V 4400 3000 50  0001 C CNN
-F 2 "Sukko:LoosePads-4" H 4400 3300 50  0001 C CNN
+F 2 "Open2327RomAdapter:LoosePads-4" H 4400 3300 50  0001 C CNN
 F 3 "" H 4400 3300 50  0001 C CNN
 	1    4400 3300
