File: Open2327RomAdapter.sch (KiCad schematic (older format))
At the start: 6 parts, among them P1 CONN_01X04, U1 2364, U2 27128

Commit message: Move solderable pads to 0.1" pitch and drill a hole through them Also port to Kicad 5 and use builtin components/footprints
Parts:
- removed P1: CONN_01X04, Open2327RomAdapter:LoosePads-4, symbol Conn_01x04
- removed R1, R2, R3: 10K, Resistors_SMD:R_0805_HandSoldering, symbol R
- removed U1: 2364, Open2327RomAdapter:DIP-24_W15.24mm-Notch, symbol 2364
- removed U2: 27128, Open2327RomAdapter:DIP-28_W15.24mm-Notch, symbol 27128
- added P1: Conn_01x04, Open2327RomAdapter:Solderable_PinHeader_1x04, symbol Connector_Generic:Conn_01x04
- added P99: OSHW_LOGO, Symbol:OSHW-Logo2_7.3x6mm_Copper, symbol conn:CONN_1
- added R1, R2, R3: 10k, Resistor_SMD:R_0805_2012Metric_Pad1.15x1.40mm_HandSolder, symbol Device:R
- added U1: 2364, Open2327RomAdapter:DIP-24_W15.24mm-Notch, symbol 2364:2364
- added U2: 27128, Open2327RomAdapter:DIP-28_W15.24mm-Notch, symbol Memory_EPROM:27128
Connections:
- wire segments 111 -> 123
- no-connect marks 0 -> 1
